Commit message: Added dual ur5 simulator

File: husky_gazebo/urdf/husky.gazebo.xacro (robot description, xacro)
@@ -30,10 +30,6 @@
         <bodyName>base_link</bodyName>
         <topicName>imu/data</topicName>
-        <accelDrift>0.005 0.005 0.005</accelDrift>
-        <accelGaussianNoise>0.005 0.005 0.005</accelGaussianNoise>
-        <rateDrift>0.005 0.005 0.005 </rateDrift>
-        <rateGaussianNoise>0.005 0.005 0.005 </rateGaussianNoise>
-        <headingDrift>0.005</headingDrift>
-        <headingGaussianNoise>0.005</headingGaussianNoise>
+        <serviceName>imu_service</serviceName>
+        <gaussianNoise>0.0</gaussianNoise>
       </plugin>
     </gazebo>
@@ -77,4 +73,98 @@
       </gazebo>
     </xacro:if>
+    <xacro:if value="$(arg robotiq_grippers_enabled)">
+        <gazebo>
+	    <plugin name="robotiq_left_hand_plugin" filename="libRobotiqHandPlugin.so">
+	      <side>left</side>
+	      <kp_position>5.0</kp_position>
+	      <kd_position>0.5</kd_position>
+	     </plugin>
+        </gazebo>
+         <gazebo>
+            <plugin name="robotiq_right_hand_plugin" filename="libRobotiqHandPlugin.so">
+              <side>right</side>
+              <kp_position>5.0</kp_position>
+              <kd_position>0.5</kd_position>
+             </plugin>
+        </gazebo>
+        <gazebo reference="l_palm">
+            <material>Gazebo/Black</material>
+        </gazebo>
+        <gazebo reference="r_palm">
+            <material>Gazebo/Black</material>
+        </gazebo>
+ <gazebo reference="l_finger_1_link_0">
+            <material>Gazebo/Black</material>
+        </gazebo>
+<gazebo reference="r_finger_1_link_0">
+            <material>Gazebo/Black</material>
+        </gazebo>
+<gazebo reference="l_finger_1_link_1">
+            <material>Gazebo/Black</material>
+        </gazebo>
+<gazebo reference="r_finger_1_link_1">
+            <material>Gazebo/Black</material>
+        </gazebo>
+<gazebo reference="l_finger_1_link_2">
+            <material>Gazebo/Black</material>
+        </gazebo>
+<gazebo reference="r_finger_1_link_2">
+            <material>Gazebo/Black</material>
+        </gazebo>
+<gazebo reference="l_finger_1_link_3">
+            <material>Gazebo/Grey</material>
+        </gazebo>
+<gazebo reference="r_finger_1_link_3">
+            <material>Gazebo/Grey</material>
+        </gazebo>
+<gazebo reference="l_finger_2_link_0">
+            <material>Gazebo/Black</material>
+        </gazebo>
+<gazebo reference="r_finger_2_link_0">
+            <material>Gazebo/Black</material>
+        </gazebo>
+<gazebo reference="l_finger_2_link_1">
+            <material>Gazebo/Black</material>
+        </gazebo>
+<gazebo reference="r_finger_2_link_1">
+            <material>Gazebo/Black</material>
+        </gazebo>
+<gazebo reference="l_finger_2_link_2">
+            <material>Gazebo/Black</material>
+        </gazebo>
+<gazebo reference="r_finger_2_link_2">
+            <material>Gazebo/Black</material>
+        </gazebo>
+<gazebo reference="l_finger_2_link_3">
+            <material>Gazebo/Grey</material>
+        </gazebo>
+<gazebo reference="r_finger_2_link_3">
+            <material>Gazebo/Grey</material>
+        </gazebo>
+<gazebo reference="l_finger_middle_link_0">
+            <material>Gazebo/Black</material>
+        </gazebo>
+<gazebo reference="r_finger_middle_link_0">
+            <material>Gazebo/Black</material>
+        </gazebo>
+<gazebo reference="l_finger_middle_link_1">
+            <material>Gazebo/Black</material>
+        </gazebo>
+<gazebo reference="r_finger_middle_link_1">
+            <material>Gazebo/Black</material>
+        </gazebo>
+<gazebo reference="l_finger_middle_link_2">
+            <material>Gazebo/Black</material>
+        </gazebo>
+<gazebo reference="r_finger_middle_link_2">
+            <material>Gazebo/Black</material>
+        </gazebo>
+<gazebo reference="l_finger_middle_link_3">
+            <material>Gazebo/Grey</material>
+        </gazebo>
+<gazebo reference="r_finger_middle_link_3">
+            <material>Gazebo/Grey</material>
+        </gazebo>
+    </xacro:if>
     <xacro:if value="$(arg kinect_enabled)">
       <xacro:kinect_camera_gazebo prefix="camera"/>
